Commit message: Start base link urdf

File: models/urdf/manuel1.urdf (robot description, URDF)
Before this commit: robot manuel1, 0 links, 0 joints
Links:
- added link base_link; visual mesh filename=visual_links/base_visual.stl scale=0.001 0.001 0.001

Commit message: Set up collision; visualization works with URDF Visualizer VS code extension

File: models/urdf/manuel1.urdf (robot description, URDF)
Before this commit: robot manuel1, 1 links, 0 joints
Links:
- link base_link: geometry collision mesh filename=collision_links/base_collision.stl scale=0.001 0.001 0.001; visual mesh filename=visual_links/base_visual.stl scale=0.001 0.001 0.001

Commit message: Shoulder joint

File: models/urdf/manuel1.urdf (robot description, URDF)
Before this commit: robot manuel1, 1 links, 0 joints
Links:
- added link shoulder_link; collision mesh filename=collision_links/shoulder_collision.stl scale=0.001 0.001 0.001; visual mesh filename=visual_links/shoulder_visual.stl scale=0.001 0.001 0.001
Joints:
- added joint waist_joint: type revolute, parent base_link, child shoulder_link, origin xyz=0.0 0.0 0 rpy=0.0 0.0 0.0, axis 0 0 1, limit lower=-3.14159265 upper=3.14159265

Commit message: Upper arm URDF

File: models/urdf/manuel1.urdf (robot description, URDF)
Before this commit: robot manuel1, 2 links, 1 joints
Links:
- added link upper_arm_link; collision mesh filename=collision_links/upper_arm_collision.stl scale=0.001 0.001 0.001; visual mesh filename=visual_links/upper_arm_visual.stl scale=0.001 0.001 0.001
Joints:
- added joint shoulder_joint: type revolute, parent shoulder_link, child upper_arm_link, origin xyz=0.0 0.0 0.1307 rpy=0.0 0.0 0.0, axis 1 0 0, limit lower=-3.14159265 upper=3.14159265

Commit message: Elbow joint and forearm

File: models/urdf/manuel1.urdf (robot description, URDF)
Before this commit: robot manuel1, 3 links, 2 joints
Links:
- added link forearm_link; collision mesh filename=collision_links/forearm_collision.stl scale=0.001 0.001 0.001; visual mesh filename=visual_links/forearm_visual.stl scale=0.001 0.001 0.001
Joints:
- added joint elbow_joint: type revolute, parent upper_arm_link, child forearm_link, origin xyz=0.0 0.0 0.305 rpy=0.0 0.0 0.0, axis 1 0 0, limit lower=-3.14159265 upper=3.14159265

Commit message: Wrist 1 joint

File: models/urdf/manuel1.urdf (robot description, URDF)
Before this commit: robot manuel1, 4 links, 3 joints
Links:
- added link wrist_12_link; collision mesh filename=collision_links/wrist_12_collision.stl scale=0.001 0.001 0.001; visual mesh filename=visual_links/wrist_12_visual.stl scale=0.001 0.001 0.001
Joints:
- added joint wrist_1_joint: type revolute, parent forearm_link, child wrist_12_link, origin xyz=0.0 0.06 0.0 rpy=0.0 0.0 0.0, axis 0 0 1, limit lower=-3.14159265 upper=3.14159265

Commit message: Wrist 2 joint

File: models/urdf/manuel1.urdf (robot description, URDF)
Before this commit: robot manuel1, 5 links, 4 joints
Links:
- added link wrist_23_link; collision mesh filename=collision_links/wrist_23_collision.stl scale=0.001 0.001 0.001; visual mesh filename=visual_links/wrist_23_visual.stl scale=0.001 0.001 0.001
Joints:
- added joint wrist_2_joint: type revolute, parent wrist_12_link, child wrist_23_link, origin xyz=0.0 0.0 0.4033 rpy=0.0 0.0 0.0, axis 1 0 0, limit lower=-3.14159265 upper=3.14159265

Commit message: Wrist 3 / gripper

File: models/urdf/manuel1.urdf (robot description, URDF)
Before this commit: robot manuel1, 6 links, 5 joints
Links:
- added link gripper_link; collision mesh filename=collision_links/gripper_collision.stl scale=0.001 0.001 0.001; visual mesh filename=visual_links/gripper_visual.stl scale=0.001 0.001 0.001
Joints:
- added joint wrist_3_joint: type revolute, parent wrist_23_link, child gripper_link, origin xyz=-0.1383 0.0 0.0 rpy=0.0 0.0 0.0, axis 0 0 1, limit lower=-3.14159265 upper=3.14159265

Commit message: Change elbow and shoulder limits

File: models/urdf/manuel1.urdf (robot description, URDF)
Before this commit: robot manuel1, 7 links, 6 joints
Joints:
- joint elbow_joint: limit lower=-3.14159265 upper=3.14159265 -> lower=0.0 upper=3.14159265
- joint shoulder_joint: limit lower=-3.14159265 upper=3.14159265 -> lower=-1.57079632 upper=1.57079632
